File: pcb/tape-punch-controller.sch (KiCad schematic (older format))
At the start: 3 parts

Commit message: Version 2 PCB design (WIP)
Parts:
- added MH4: Screw_Terminal_01x01, Mounting_Holes:MountingHole_4.3mm_M4_Pad_Via, symbol Screw_Terminal_01x01
- MH1: renamed from MP1; footprint Mounting_Holes:MountingHole_4.3mm_M4_Pad -> Mounting_Holes:MountingHole_4.3mm_M4_Pad_Via
- MH2: renamed from MP2; footprint Mounting_Holes:MountingHole_4.3mm_M4_Pad -> Mounting_Holes:MountingHole_4.3mm_M4_Pad_Via
- MH3: renamed from MP3; footprint Mounting_Holes:MountingHole_4.3mm_M4_Pad -> Mounting_Holes:MountingHole_4.3mm_M4_Pad_Via
Connections:
- net GND: now also MH4.1 (Pin_1)
Changed lines of the file:
@@
 LIBS:valves
 LIBS:symbols
-LIBS:tape-punch-controller-cache
 EELAYER 25 0
 EELAYER END
@@
 $EndSheet
 $Comp
-L Screw_Terminal_01x01 MP1
+L Screw_Terminal_01x01 MH1
 U 1 1 5A3E86DB
 P 9800 4850
-F 0 "MP1" H 9800 4950 50  0000 C CNN
+F 0 "MH1" H 9800 4950 50  0000 C CNN
 F 1 "Screw_Terminal_01x01" H 9800 4750 50  0000 C CNN
-F 2 "Mounting_Holes:MountingHole_4.3mm_M4_Pad" H 9800 4850 50  0001 C CNN
+F 2 "Mounting_Holes:MountingHole_4.3mm_M4_Pad_Via" H 9800 4850 50  0001 C CNN
 F 3 "" H 9800 4850 50  0001 C CNN
 	1    9800 4850
@@
 $EndComp
 $Comp
-L Screw_Terminal_01x01 MP2
+L Screw_Terminal_01x01 MH2
 U 1 1 5A3E8774
 P 9800 5150
-F 0 "MP2" H 9800 5250 50  0000 C CNN
+F 0 "MH2" H 9800 5250 50  0000 C CNN
 F 1 "Screw_Terminal_01x01" H 9800 5050 50  0000 C CNN
-F 2 "Mounting_Holes:MountingHole_4.3mm_M4_Pad" H 9800 5150 50  0001 C CNN
+F 2 "Mounting_Holes:MountingHole_4.3mm_M4_Pad_Via" H 9800 5150 50  0001 C CNN
 F 3 "" H 9800 5150 50  0001 C CNN
 	1    9800 5150
@@
 $EndComp
 $Comp
-L Screw_Terminal_01x01 MP3
+L Screw_Terminal_01x01 MH3
 U 1 1 5A3E8794
 P 9800 5450
-F 0 "MP3" H 9800 5550 50  0000 C CNN
+F 0 "MH3" H 9800 5550 50  0000 C CNN
 F 1 "Screw_Terminal_01x01" H 9800 5350 50  0000 C CNN
-F 2 "Mounting_Holes:MountingHole_4.3mm_M4_Pad" H 9800 5450 50  0001 C CNN
+F 2 "Mounting_Holes:MountingHole_4.3mm_M4_Pad_Via" H 9800 5450 50  0001 C CNN
 F 3 "" H 9800 5450 50  0001 C CNN
 	1    9800 5450
@@
 L GND #PWR01
 U 1 1 5A3E882F
-P 9200 5500
-F 0 "#PWR01" H 9200 5250 50  0001 C CNN
-F 1 "GND" H 9200 5350 50  0000 C CNN
-F 2 "" H 9200 5500 50  0001 C CNN
-F 3 "" H 9200 5500 50  0001 C CNN
-	1    9200 5500
+P 9200 5850
+F 0 "#PWR01" H 9200 5600 50  0001 C CNN
+F 1 "GND" H 9200 5700 50  0000 C CNN
+F 2 "" H 9200 5850 50  0001 C CNN
+F 3 "" H 9200 5850 50  0001 C CNN
+	1    9200 5850
 	1    0    0    -1
 $EndComp
@@
 	9600 4850 9200 4850
 Wire Wire Line
-	9200 4850 9200 5500
+	9200 4850 9200 5850
 Wire Wire Line
 	9600 5150 9200 5150
@@
 Text Notes 9600 2700 0    60   ~ 0
 Tape punch
+$Comp
+L Screw_Terminal_01x01 MH4
+U 1 1 5A5A3E45
+P 9800 5750
+F 0 "MH4" H 9800 5850 50  0000 C CNN
+F 1 "Screw_Terminal_01x01" H 9800 5650 50  0000 C CNN
+F 2 "Mounting_Holes:MountingHole_4.3mm_M4_Pad_Via" H 9800 5750 50  0001 C CNN
+F 3 "" H 9800 5750 50  0001 C CNN
+	1    9800 5750
+	1    0    0    -1
+$EndComp
+Wire Wire Line
+	9200 5750 9600 5750
+Connection ~ 9200 5750
 $EndSCHEMATC

Commit message: Finish draft of second version of PCB
Parts:
- removed MH4: Screw_Terminal_01x01, Mounting_Holes:MountingHole_4.3mm_M4_Pad_Via, symbol Screw_Terminal_01x01
- MH1, MH2, MH3: footprint Mounting_Holes:MountingHole_4.3mm_M4_Pad_Via -> Mounting_Holes:MountingHole_4.3mm_M4_Pad
Changed lines of the file:
@@
 LIBS:valves
 LIBS:symbols
+LIBS:tape-punch-controller-cache
 EELAYER 25 0
 EELAYER END
@@
 F 0 "MH1" H 9800 4950 50  0000 C CNN
 F 1 "Screw_Terminal_01x01" H 9800 4750 50  0000 C CNN
-F 2 "Mounting_Holes:MountingHole_4.3mm_M4_Pad_Via" H 9800 4850 50  0001 C CNN
+F 2 "Mounting_Holes:MountingHole_4.3mm_M4_Pad" H 9800 4850 50  0001 C CNN
 F 3 "" H 9800 4850 50  0001 C CNN
 	1    9800 4850
@@
 F 0 "MH2" H 9800 5250 50  0000 C CNN
 F 1 "Screw_Terminal_01x01" H 9800 5050 50  0000 C CNN
-F 2 "Mounting_Holes:MountingHole_4.3mm_M4_Pad_Via" H 9800 5150 50  0001 C CNN
+F 2 "Mounting_Holes:MountingHole_4.3mm_M4_Pad" H 9800 5150 50  0001 C CNN
 F 3 "" H 9800 5150 50  0001 C CNN
 	1    9800 5150
@@
 F 0 "MH3" H 9800 5550 50  0000 C CNN
 F 1 "Screw_Terminal_01x01" H 9800 5350 50  0000 C CNN
-F 2 "Mounting_Holes:MountingHole_4.3mm_M4_Pad_Via" H 9800 5450 50  0001 C CNN
+F 2 "Mounting_Holes:MountingHole_4.3mm_M4_Pad" H 9800 5450 50  0001 C CNN
 F 3 "" H 9800 5450 50  0001 C CNN
 	1    9800 5450
@@
 L GND #PWR01
 U 1 1 5A3E882F
-P 9200 5850
-F 0 "#PWR01" H 9200 5600 50  0001 C CNN
-F 1 "GND" H 9200 5700 50  0000 C CNN
-F 2 "" H 9200 5850 50  0001 C CNN
-F 3 "" H 9200 5850 50  0001 C CNN
-	1    9200 5850
+P 9200 5550
+F 0 "#PWR01" H 9200 5300 50  0001 C CNN
+F 1 "GND" H 9200 5400 50  0000 C CNN
+F 2 "" H 9200 5550 50  0001 C CNN
+F 3 "" H 9200 5550 50  0001 C CNN
+	1    9200 5550
 	1    0    0    -1
 $EndComp
@@
 	9600 4850 9200 4850
 Wire Wire Line
-	9200 4850 9200 5850
+	9200 4850 9200 5550
 Wire Wire Line
 	9600 5150 9200 5150
@@
 Text Notes 9600 2700 0    60   ~ 0
 Tape punch
-$Comp
-L Screw_Terminal_01x01 MH4
-U 1 1 5A5A3E45
-P 9800 5750
-F 0 "MH4" H 9800 5850 50  0000 C CNN
-F 1 "Screw_Terminal_01x01" H 9800 5650 50  0000 C CNN
-F 2 "Mounting_Holes:MountingHole_4.3mm_M4_Pad_Via" H 9800 5750 50  0001 C CNN
-F 3 "" H 9800 5750 50  0001 C CNN
-	1    9800 5750
-	1    0    0    -1
-$EndComp
-Wire Wire Line
-	9200 5750 9600 5750
-Connection ~ 9200 5750
 $EndSCHEMATC
