File: pcb/solenoid-drivers.sch (KiCad schematic (older format))
At the start: 62 parts, among them Q1 IRLZ44N, Q10 IRLML0060, Q2 IRLZ44N, Q3 IRLZ44N, Q4 IRLZ44N, Q5 IRLZ44N, Q6 IRLZ44N, Q7 IRLZ44N, Q8 IRLZ44N, Q9 IRLZ44N

Commit message: Version 2 PCB design (WIP)
Parts:
- removed Q1, Q2, Q3, Q4, Q5, Q6, Q7, Q8, Q9: IRLZ44N, TO_SOT_Packages_THT:TO-220-3_Vertical, symbol Q_NMOS_GDS
- added Q1, Q2, Q3, Q4, Q5, Q6, Q7, Q8, Q9: IRLML0060, TO_SOT_Packages_SMD:SOT-23_Handsoldering, symbol Q_NMOS_GSD
- Q10: footprint (none) -> TO_SOT_Packages_SMD:SOT-23_Handsoldering
- renumbered R6 to R11, R7 to R12, R8 to R13, R15 to R14, R16 to R15, R17 to R16, R18 to R17, R5 to R18, R9 to R19, R19 to R20, R11 to R21, R12 to R22, R13 to R23, R20 to R24, R21 to R25, R22 to R26, R23 to R27, R10 to R28, R14 to R29, R24 to R30, R25 to R33, TP5 to TP14, TP6 to TP15, TP7 to TP16, TP8 to TP17, TP9 to TP18, TP10 to TP19, TP11 to TP20, TP12 to TP21, TP13 to TP22, TP14 to TP23, TP15 to TP24, TP16 to TP25, TP17 to TP26, TP18 to TP27, TP19 to TP28, TP20 to TP29, TP21 to TP30, TP22 to TP31, TP23 to TP32, TP24 to TP33, TP25 to TP34, TP26 to TP35, TP27 to TP36, TP28 to TP37, TP29 to TP38, TP30 to TP39, TP31 to TP40, TP32 to TP41, TP33 to TP42, TP34 to TP43, TP35 to TP44
