File: pcb/tape-punch-connector.sch (KiCad schematic (older format))
At the start: 11 parts, among them J1 DB25_Male_MountingHoles

Commit message: Version 2 PCB design (WIP)
Parts:
- removed J1: DB25_Male_MountingHoles, local:NORCOMP_182-025-113R171, symbol DB25_Male_MountingHoles
- added J1: Conn_01x06, Local:Amphenol_T821106A1S100CEU, symbol Conn_01x06
- added J2: Conn_01x09, Local:Weidmuller_1234610000, symbol Conn_01x09
- renumbered C1 to C12, C2 to C13, R3 to R34, R4 to R35, R1 to R36, R2 to R37, TP3 to TP45, TP4 to TP46, TP1 to TP47, TP2 to TP48
Connections:
- net labels removed: +28V, TP_EARTH
- wire segments 42 -> 56
- no-connect marks 4 -> 0
Other:
- note added: "Each pin on J2 is wired to the pin of the\nsame number on the DB25 (tape punch)\nconnector mounted on the chassis.\nThese are the negative ends of the nine\nsolenoids. The positive ends are connected\nto the 28V rail inside the tape punch, which\nitself is directly connected to the PSU."
- note added: "LOW_TAPE_RAW/NO_TAPE_RAW are normally connected\nto ground by their respective switches. If a low tape or\nno tape condition occurs, the switch disconnects, allowing\nthe corresponding _RAW signal to be pulled high by the\n10k resistor.\n\nEach switch is debounced with an RC filter."
- note added: "Miscellaneous low-current signals for the tape punch.\n\nENABLE_RELAY is the negative end of the relay that\nconnects power to the motor and solenoids. The\npositive end of this relay is tied to the 28V supply\ninside the tape punch.\n\nThe feedback coil is connected between SYNC_COIL+\nand SYNC_COIL-.\n\nLOW_TAPE_RAW and NO_TAPE_RAW connect to the\ntwo switches inside the tape punch; see the com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"
- note added: "Tape punch cable pinout:\n\nTP pin 1 -- J2 pin 1 (code sol 1)\nTP pin 2 -- J2 pin 2 (code sol 2)\nTP pin 3 -- J2 pin 3 (code sol 3)\nTP pin 4 -- J2 pin 4 (code sol 4)\nTP pin 5 -- J2 pin 5 (code sol 5)\nTP pin 6 -- J2 pin 6 (code sol 6)\nTP pin 7 -- J2 pin 7 (code sol 7)\nTP pin 8 -- J2 pin 8 (code sol 0)\nTP pin 9 -- J2 pin 9 (feed sol)\nTP pin 10 -- PSU 28VDC output\nTP pin 11 -- earth (tape pu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"
- note removed: "LOW_TAPE_RAW/NO_TAPE_RAW are\nnormally held high, and are driven\nlow when the corresponding switches\ndetect that reel is not low on tape or\nthat there is tape present. Each switch\nis debounced using an RC filter."
- note removed: "Pinout description:"
- note removed: "Pins 1-9 are the negative sides of the\nsolenoids. The positive sides are\nconnected to the 28V supply rail via\npins 10, 18, 19 and 23.\n\nPin 25 is the negative side of the coil\nof the power relay. The positive side is\nlikewise connected to the 28V rail.\n\nPins 12 and 24 are connected to the\nfeedback coil.\n\nPins 13, 14 and 15 are connected to\nthe tape detection switch, located just\nnext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"
- moved on the sheet: C12, C13, R34, R35, R36, R37, TP45, TP46, TP47, TP48
